File: power_distribution_board/HW/PCB/francor_power_distribution.kicad_pcb (KiCad board)
At the start: 2 copper layers, 49.8 x 92.7 mm, 20 parts, among them J1 Conn_01x04_3.81, J10 Conn_01x04_3.81, J11 Conn_01x04_3.81, J12 Conn_01x04_3.81, J13 ESQ-102-24-T-D, J14 ESQ-102-24-T-D, J15 ESQ-102-24-T-D, J16 ESQ-102-24-T-D, J2 Conn_01x04_3.81, J3 Conn_01x04_3.81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

Commit message: Added text to PCBs
Other:
- board text added: "Power Distribution Board FRANCOR e.V."
Changed lines of the file:
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@@
   (general
     (thickness 1.6)
-    (drawings 8)
+    (drawings 9)
     (tracks 98)
     (zones 0)
@@
   )
   (setup
-    (last_trace_width 4)
+    (last_trace_width 1.27)
     (user_trace_width 1.27)
     (user_trace_width 2)
@@
       (net 4 /GND))
   )
+  (gr_text "Power Distribution Board\nFRANCOR e.V." (at 140.97 92.71 90) (layer F.SilkS)
+    (effects (font (size 1.5 1.5) (thickness 0.3)))
+  )
   (target plus (at 116.078 137.16) (size 5) (width 0.05) (layer Edge.Cuts))
